Commit message: feat(manipulator): raise arm joint effort, add sim-only wrist roll + tapered jaws

File: rosbot_description/urdf/open_manipulator/body.xacro (robot description, xacro)
@@ -6,7 +6,97 @@
                     rpy:='0.0 0.0 0.0'
                     namespace:=''
-                    prefix:=''">
+                    prefix:=''
+                    wrist_roll:='false'
+                    taper_jaws:='false'">
+    <!-- Optional wrist roll about the tool axis, inserted between link5 and the
+         gripper. Off by default and only switched on for simulation: the real
+         OpenMANIPULATOR-X is 4-DOF with no such servo, and the Dynamixel driver
+         is pinned to number_of_joints=5 (4 arm plus gripper), so a fifth arm
+         joint on the hardware path would not map to anything. -->
+    <xacro:property name="roll_on" value="${wrist_roll in ['true', 'True', True]}"/>
+    <xacro:property name="gripper_parent" value="${prefix + ('link5_roll' if roll_on else 'link5')}"/>
+    <!-- Tapered V jaws, shaped for a shuttlecock lying on its side.
+         The stock jaws are flat parallel plates, so against a cone they touch
+         only at the widest station: point contact, and the cone pivots and
+         rolls straight out. Each jaw here is two pads instead:
+           * both pads pitched by the cone's 18 deg half-angle, so the faces
+             stay parallel to the flank along their whole length rather than
+             meeting it at a point,
+           * the pair splayed into a 120 deg included V whose valley runs along
+             the cone axis, giving two contact lines per side that box the
+             object in and stop it rolling.
+         Collision is boxes, deliberately. A single notched mesh would be run
+         through a convex hull by the physics engine, which fills the notch in
+         and throws away the part that does the work. -->
+    <xacro:property name="taper_on" value="${taper_jaws in ['true', 'True', True]}"/>
+    <xacro:property name="cone_half_angle" value="0.3142"/>   <!-- 18 deg -->
+    <xacro:property name="v_half_angle" value="1.0472"/>      <!-- 120 deg included -->
+    <xacro:property name="pad_x" value="0.030"/>              <!-- along the blade -->
+    <xacro:property name="pad_t" value="0.005"/>              <!-- thickness -->
+    <xacro:property name="pad_z" value="0.075"/>              <!-- along the cone axis -->
+    <xacro:property name="pad_centre_x" value="0.045"/>       <!-- matches GRASP_OFFSET -->
+    <xacro:property name="pad_split" value="0.016"/>          <!-- V half-width -->
+    <!-- Kept small so the jaws still open wider than the 65 mm skirt: the gap
+         is 2*(0.021 + q - inset), which at the open stop leaves a few mm a
+         side to drop over the object instead of knocking it. -->
+    <xacro:property name="pad_inset" value="0.001"/>
+    <!-- One pad. side=+1 for the left jaw, -1 for the right. lobe=+1/-1 picks
+         which half of the V. -->
+    <xacro:macro name="taper_pad" params="side lobe">
+      <collision>
+        <origin xyz="${pad_centre_x + lobe * pad_split} ${-side * pad_inset} 0"
+                rpy="${side * cone_half_angle} 0 ${side * lobe * (v_half_angle / 2)}"/>
+        <geometry>
+          <box size="${pad_x} ${pad_t} ${pad_z}"/>
+        </geometry>
+        <surface>
+          <friction><ode><mu>1.2</mu><mu2>1.2</mu2></ode></friction>
+        </surface>
+      </collision>
+      <visual>
+        <origin xyz="${pad_centre_x + lobe * pad_split} ${-side * pad_inset} 0"
+                rpy="${side * cone_half_angle} 0 ${side * lobe * (v_half_angle / 2)}"/>
+        <geometry>
+          <box size="${pad_x} ${pad_t} ${pad_z}"/>
+        </geometry>
+        <material name="jaw_grey">
+          <color rgba="0.25 0.25 0.28 1"/>
+        </material>
+      </visual>
+    </xacro:macro>
+    <!-- Backing plate carrying the pads back to the joint. -->
+    <xacro:macro name="taper_spine" params="side">
+      <collision>
+        <origin xyz="0.030 ${-side * 0.001} 0" rpy="0 0 0"/>
+        <geometry>
+          <box size="0.060 0.008 0.030"/>
+        </geometry>
+      </collision>
+      <visual>
+        <origin xyz="0.030 ${-side * 0.001} 0" rpy="0 0 0"/>
+        <geometry>
+          <box size="0.060 0.008 0.030"/>
+        </geometry>
+        <material name="jaw_grey">
+          <color rgba="0.25 0.25 0.28 1"/>
+        </material>
+      </visual>
+    </xacro:macro>
     <xacro:property name="meshes_dir" value="package://open_manipulator_description/meshes/open_manipulator_x"/>
     <xacro:property name="link1_length" value="0.06"/>
+    <!-- Stall torque in Nm of the XM430-W350 servos used by the
+         OpenMANIPULATOR-X at 12 V. The joints previously carried a placeholder
+         effort of 1, below what joint2 needs just to hold the arm out. It
+         settled about 0.2 rad short of any commanded reach-down pose, leaving
+         the gripper roughly 30 mm high. The prismatic gripper joints are in
+         newtons, not Nm, and are set separately below. -->
+    <xacro:property name="servo_effort" value="4.1"/>
+    <!-- Grip force in N for the prismatic finger joints, left at the original
+         value. In free space the fingers track every commanded position
+         exactly, including the fully closed -0.009, so 1 N is not the limit on
+         normal operation. Raising it to 15 N was tried and did not help the
+         fingers close while in contact with the target, so it was reverted
+         rather than left as an unexplained deviation. -->
+    <xacro:property name="gripper_effort" value="1"/>
     <xacro:if value="${parent_link != ''}">
       <joint name="${prefix}${parent_link}_to_link1" type="fixed">
@@ -50,5 +140,5 @@
       <origin xyz="0.0 0.0 0.017" rpy="0 0 0"/>
       <axis xyz="0 0 1"/>
-      <limit velocity="4.8" effort="1" lower="${-4/5*pi}" upper="${pi}" />
+      <limit velocity="4.8" effort="${servo_effort}" lower="${-4/5*pi}" upper="${pi}" />
       <dynamics damping="0.1"/>
     </joint>
@@ -82,5 +172,5 @@
       <origin xyz="0.0 0.0 0.0595" rpy="0 0 0"/>
       <axis xyz="0 1 0"/>
-      <limit velocity="4.8" effort="1" lower="${-pi/2}" upper="${pi/2}" />
+      <limit velocity="4.8" effort="${servo_effort}" lower="${-pi/2}" upper="${pi/2}" />
       <dynamics damping="0.1"/>
     </joint>
@@ -114,5 +204,5 @@
       <origin xyz="0.024 0 0.128" rpy="0 0 0"/>
       <axis xyz="0 1 0"/>
-      <limit velocity="4.8" effort="1" lower="${-1.5}" upper="${1.4}" />
+      <limit velocity="4.8" effort="${servo_effort}" lower="${-1.5}" upper="${1.4}" />
       <dynamics damping="0.1"/>
     </joint>
@@ -146,5 +236,5 @@
       <origin xyz="0.124 0.0 0.0" rpy="0 0 0"/>
       <axis xyz="0 1 0"/>
-      <limit velocity="4.8" effort="1" lower="${-1.7}" upper="${1.97}" />
+      <limit velocity="4.8" effort="${servo_effort}" lower="${-1.7}" upper="${1.97}" />
       <dynamics damping="0.1"/>
     </joint>
@@ -173,28 +263,58 @@
       </inertial>
     </link>
+    <!-- Wrist roll. Axis 1 0 0 is link5's own x, which is the tool axis the
+         gripper points along, so this spins the jaws about their approach
+         direction without moving the grasp point. That keeps the position
+         kinematics of joints 1-4 untouched. -->
+    <xacro:if value="${roll_on}">
+      <joint name="${prefix}joint5" type="revolute">
+        <parent link="${prefix}link5"/>
+        <child link="${prefix}link5_roll"/>
+        <origin xyz="0 0 0" rpy="0 0 0"/>
+        <axis xyz="1 0 0"/>
+        <limit velocity="4.8" effort="${servo_effort}" lower="${-pi}" upper="${pi}" />
+        <dynamics damping="0.1"/>
+      </joint>
+      <link name="${prefix}link5_roll">
+        <inertial>
+          <origin xyz="0 0 0" />
+          <mass value="1.0e-03" />
+          <inertia ixx="1.0e-06" ixy="0.0" ixz="0.0"
+                   iyy="1.0e-06" iyz="0.0"
+                   izz="1.0e-06" />
+        </inertial>
+      </link>
+    </xacro:if>
     <joint name="${prefix}gripper_left_joint" type="prismatic">
-      <parent link="${prefix}link5"/>
+      <parent link="${gripper_parent}"/>
       <child link="${prefix}gripper_left_link"/>
       <origin xyz="0.0817 0.021 0.0" rpy="0 0 0"/>
       <axis xyz="0 1 0"/>
-      <limit velocity="4.8" effort="1" lower="-0.010" upper="0.019" />
+      <limit velocity="4.8" effort="${gripper_effort}" lower="-0.010" upper="0.019" />
       <dynamics damping="0.1"/>
     </joint>
     <link name="${prefix}gripper_left_link">
-      <visual>
-        <origin xyz="0 0 0" rpy="0 0 0"/>
-        <geometry>
-          <mesh filename="${meshes_dir}/gripper_left_palm.stl" scale="0.001 0.001 0.001"/>
-        </geometry>
-        <material name="grey">
-          <color rgba="0.2 0.2 0.2 1"/>
-        </material>
-      </visual>
-      <collision>
-        <origin xyz="0 0 0" rpy="0 0 0"/>
-        <geometry>
-          <mesh filename="${meshes_dir}/gripper_left_palm.stl" scale="0.001 0.001 0.001"/>
-        </geometry>
-      </collision>
+      <xacro:if value="${taper_on}">
+        <xacro:taper_spine side="1"/>
+        <xacro:taper_pad side="1" lobe="1"/>
+        <xacro:taper_pad side="1" lobe="-1"/>
+      </xacro:if>
+      <xacro:unless value="${taper_on}">
+        <visual>
+          <origin xyz="0 0 0" rpy="0 0 0"/>
+          <geometry>
+            <mesh filename="${meshes_dir}/gripper_left_palm.stl" scale="0.001 0.001 0.001"/>
+          </geometry>
+          <material name="grey">
+            <color rgba="0.2 0.2 0.2 1"/>
+          </material>
+        </visual>
+        <collision>
+          <origin xyz="0 0 0" rpy="0 0 0"/>
+          <geometry>
+            <mesh filename="${meshes_dir}/gripper_left_palm.stl" scale="0.001 0.001 0.001"/>
+          </geometry>
+        </collision>
+      </xacro:unless>
       <inertial>
         <origin xyz="0 0 0" />
@@ -206,28 +326,35 @@
     </link>
     <joint name="${prefix}gripper_right_joint" type="prismatic">
-      <parent link="${prefix}link5"/>
+      <parent link="${gripper_parent}"/>
       <child link="${prefix}gripper_right_link"/>
       <origin xyz="0.0817 -0.021 0" rpy="0 0 0"/>
       <axis xyz="0 -1 0"/>
-      <limit velocity="4.8" effort="1" lower="-0.010" upper="0.019" />
+      <limit velocity="4.8" effort="${gripper_effort}" lower="-0.010" upper="0.019" />
       <mimic joint="${prefix}gripper_left_joint" multiplier="1"/>
       <dynamics damping="0.1"/>
     </joint>
     <link name="${prefix}gripper_right_link">
-      <visual>
-        <origin xyz="0 0 0" rpy="0 0 0"/>
-        <geometry>
-          <mesh filename="${meshes_dir}/gripper_right_palm.stl" scale="0.001 0.001 0.001"/>
-        </geometry>
-        <material name="grey">
-          <color rgba="0.2 0.2 0.2 1"/>
-        </material>
-      </visual>
-      <collision>
-        <origin xyz="0 0 0" rpy="0 0 0"/>
-        <geometry>
-          <mesh filename="${meshes_dir}/gripper_right_palm.stl" scale="0.001 0.001 0.001"/>
-        </geometry>
-      </collision>
+      <xacro:if value="${taper_on}">
+        <xacro:taper_spine side="-1"/>
+        <xacro:taper_pad side="-1" lobe="1"/>
+        <xacro:taper_pad side="-1" lobe="-1"/>
+      </xacro:if>
+      <xacro:unless value="${taper_on}">
+        <visual>
+          <origin xyz="0 0 0" rpy="0 0 0"/>
+          <geometry>
+            <mesh filename="${meshes_dir}/gripper_right_palm.stl" scale="0.001 0.001 0.001"/>
+          </geometry>
+          <material name="grey">
+            <color rgba="0.2 0.2 0.2 1"/>
+          </material>
+        </visual>
+        <collision>
+          <origin xyz="0 0 0" rpy="0 0 0"/>
+          <geometry>
+            <mesh filename="${meshes_dir}/gripper_right_palm.stl" scale="0.001 0.001 0.001"/>
+          </geometry>
+        </collision>
+      </xacro:unless>
       <inertial>
         <origin xyz="0 0 0" />
@@ -239,5 +366,5 @@
     </link>
     <joint name="${prefix}end_effector_joint" type="fixed">
-      <parent link="${prefix}link5"/>
+      <parent link="${gripper_parent}"/>
       <child link="${prefix}end_effector_link"/>
       <origin xyz="0.126 0.0 0.0" rpy="0 0 0"/>

File: rosbot_description/urdf/open_manipulator/open_manipulator_x_macro.xacro (robot description, xacro)
@@ -10,5 +10,8 @@
                     mock_sensor_commands:=false
                     use_sim:=false
+                    wrist_roll:='false'
+                    taper_jaws:='false'
                     port_name:='/dev/ttyUSB0'">
+    <xacro:property name="roll_on" value="${wrist_roll in ['true', 'True', True]}"/>
     <!-- PROPERTIES -->
     <xacro:property name="prefix" value="${device_namespace + '_' if device_namespace != '' else ''}" />
@@ -22,5 +25,7 @@
       parent_link="${parent_link}"
       xyz="${xyz}"
-      rpy="${rpy}" />
+      rpy="${rpy}"
+      wrist_roll="${wrist_roll}"
+      taper_jaws="${taper_jaws}" />
     <!-- ROS2 CONTROL PLUGINS -->
     <xacro:ros2_control.open_manipulator_x_system
@@ -31,4 +36,21 @@
       mock_sensor_commands="${mock_sensor_commands}"
       port_name="${port_name}" />
+    <!-- Wrist roll gets its own ros2_control system rather than being added to
+         the upstream OpenManipulatorXSystem block, which lives in
+         open_manipulator_description and hardcodes joints 1-4 plus the gripper.
+         Keeping it separate avoids forking that upstream file. Simulation only,
+         so the Dynamixel hardware path never sees this joint. -->
+    <xacro:if value="${roll_on}">
+      <ros2_control name="WristRollSystem" type="system">
+        <hardware>
+          <plugin>gz_ros2_control/GazeboSimSystem</plugin>
+        </hardware>
+        <joint name="${prefix}joint5">
+          <command_interface name="position"/>
+          <state_interface name="position"/>
+          <state_interface name="velocity"/>
+        </joint>
+      </ros2_control>
+    </xacro:if>
     <!-- GAZEBO PLUGINS -->
     <xacro:if value="${use_sim}">

File: rosbot_description/urdf/rosbot_xl.urdf.xacro (robot description, xacro)
@@ -33,4 +33,6 @@
       device_namespace="''"
       use_sim="$(arg use_sim)"
+      wrist_roll="$(arg use_sim)"
+      taper_jaws="$(arg use_sim)"
       port_name="$(arg manipulator_serial_port)"/>
   </xacro:if>

Commit message: fix(manipulator): widen tapered jaws, move arm to chassis front, relocate lidar

File: rosbot_description/urdf/open_manipulator/body.xacro (robot description, xacro)
@@ -37,8 +37,15 @@
     <xacro:property name="pad_centre_x" value="0.045"/>       <!-- matches GRASP_OFFSET -->
     <xacro:property name="pad_split" value="0.016"/>          <!-- V half-width -->
-    <!-- Kept small so the jaws still open wider than the 65 mm skirt: the gap
-         is 2*(0.021 + q - inset), which at the open stop leaves a few mm a
-         side to drop over the object instead of knocking it. -->
-    <xacro:property name="pad_inset" value="0.001"/>
+    <!-- Pads sit outboard of the finger frame. The naive gap of
+         2*(0.021 + q - inset) counts only the pad's 5 mm thickness and is
+         badly wrong here, because each pad is rotated 60 deg about z and 18 deg
+         about x, which swings its 30 mm and 75 mm dimensions into the closing
+         direction and brings the corners ~20 mm further in. At inset +0.001 the
+         real opening was 34.8 mm against a 65 mm skirt, so the jaws could never
+         fit around the object and knocked it aside on every approach.
+         At -0.019 the measured opening is 74.8 mm, clearing the 65 mm rim, and
+         22.8 mm closed, so the cork can still be pinched. Recompute the corner
+         extents if the pad size or either angle changes. -->
+    <xacro:property name="pad_inset" value="-0.019"/>
     <!-- One pad. side=+1 for the left jaw, -1 for the right. lobe=+1/-1 picks
          which half of the V. -->
@@ -68,5 +75,5 @@
     <xacro:macro name="taper_spine" params="side">
       <collision>
-        <origin xyz="0.030 ${-side * 0.001} 0" rpy="0 0 0"/>
+        <origin xyz="0.030 ${-side * pad_inset} 0" rpy="0 0 0"/>
         <geometry>
           <box size="0.060 0.008 0.030"/>
@@ -74,5 +81,5 @@
       </collision>
       <visual>
-        <origin xyz="0.030 ${-side * 0.001} 0" rpy="0 0 0"/>
+        <origin xyz="0.030 ${-side * pad_inset} 0" rpy="0 0 0"/>
         <geometry>
           <box size="0.060 0.008 0.030"/>

File: rosbot_description/urdf/rosbot_xl.urdf.xacro (robot description, xacro)
@@ -30,5 +30,5 @@
     <xacro:open_manipulator_x
       parent_link="'cover_link'"
-      xyz="-0.11 0.0 0.0"
+      xyz="0.065 0.0 0.0"
       device_namespace="''"
       use_sim="$(arg use_sim)"

Commit message: feat(manipulator): fit the CAD claw, and let the jaws close fully

File: rosbot_description/urdf/open_manipulator/body.xacro (robot description, xacro)
@@ -14,4 +14,5 @@
          is pinned to number_of_joints=5 (4 arm plus gripper), so a fifth arm
          joint on the hardware path would not map to anything. -->
+    <xacro:include filename="$(find rosbot_description)/urdf/open_manipulator/claw_collision.xacro"/>
     <xacro:property name="roll_on" value="${wrist_roll in ['true', 'True', True]}"/>
     <xacro:property name="gripper_parent" value="${prefix + ('link5_roll' if roll_on else 'link5')}"/>
@@ -48,4 +49,12 @@
          extents if the pad size or either angle changes. -->
     <xacro:property name="pad_inset" value="-0.019"/>
+    <!-- Finger travel. The stock jaws keep their original lower stop of
+         negative 0.010. The CAD claw needs more. Its grip surfaces sit 2 mm
+         outboard of the finger frame, so the gap is 2x(0.021 + q + 0.002) and
+         the old stop bottomed out at 26 mm, wide enough for the 26 mm cork to
+         slip straight through, which is what let the shuttlecock escape.
+         Negative 0.023 brings the claws to touching while leaving the open gap
+         at 84 mm, since only the lower stop moves. -->
+    <xacro:property name="gripper_lower" value="${-0.023 if taper_on else -0.010}"/>
     <!-- One pad. side=+1 for the left jaw, -1 for the right. lobe=+1/-1 picks
          which half of the V. -->
@@ -298,12 +307,20 @@
       <origin xyz="0.0817 0.021 0.0" rpy="0 0 0"/>
       <axis xyz="0 1 0"/>
-      <limit velocity="4.8" effort="${gripper_effort}" lower="-0.010" upper="0.019" />
+      <limit velocity="4.8" effort="${gripper_effort}" lower="${gripper_lower}" upper="0.019" />
       <dynamics damping="0.1"/>
     </joint>
     <link name="${prefix}gripper_left_link">
       <xacro:if value="${taper_on}">
-        <xacro:taper_spine side="1"/>
-        <xacro:taper_pad side="1" lobe="1"/>
-        <xacro:taper_pad side="1" lobe="-1"/>
+        <visual>
+          <origin xyz="0 0.002 0" rpy="${-pi/2} 0 ${pi/2}"/>
+          <geometry>
+            <mesh filename="package://rosbot_description/meshes/rosbot_xl/claw/Gripper-Left.stl"
+                  scale="0.001 0.001 0.001"/>
+          </geometry>
+          <material name="claw_grey">
+            <color rgba="0.25 0.25 0.28 1"/>
+          </material>
+        </visual>
+        <xacro:claw_collision_left/>
       </xacro:if>
       <xacro:unless value="${taper_on}">
@@ -337,5 +354,5 @@
       <origin xyz="0.0817 -0.021 0" rpy="0 0 0"/>
       <axis xyz="0 -1 0"/>
-      <limit velocity="4.8" effort="${gripper_effort}" lower="-0.010" upper="0.019" />
+      <limit velocity="4.8" effort="${gripper_effort}" lower="${gripper_lower}" upper="0.019" />
       <mimic joint="${prefix}gripper_left_joint" multiplier="1"/>
       <dynamics damping="0.1"/>
@@ -343,7 +360,15 @@
     <link name="${prefix}gripper_right_link">
       <xacro:if value="${taper_on}">
-        <xacro:taper_spine side="-1"/>
-        <xacro:taper_pad side="-1" lobe="1"/>
-        <xacro:taper_pad side="-1" lobe="-1"/>
+        <visual>
+          <origin xyz="0 -0.002 0" rpy="${-pi/2} 0 ${pi/2}"/>
+          <geometry>
+            <mesh filename="package://rosbot_description/meshes/rosbot_xl/claw/Gripper-Right.stl"
+                  scale="0.001 0.001 0.001"/>
+          </geometry>
+          <material name="claw_grey">
+            <color rgba="0.25 0.25 0.28 1"/>
+          </material>
+        </visual>
+        <xacro:claw_collision_right/>
       </xacro:if>
       <xacro:unless value="${taper_on}">
